File: board/flippie.sch (EAGLE design)
At the start: 28 parts, among them J1 INT_3V3, U1 FPF2702MX, U10 ULN2803ADW, U11 TD62783AP, U12 TD62783AP, U13 TD62783AP, U14 ULN2803ADW, U2 SN74AHC595D, U3 SN74AHC595D, U4 SN74AHC595D, U5 SN74AHC595D, U6 SN74AHC595D, U7 SN74AHC595D, U8 SN74AHC595D, U9 ULN2803ADW, X1 PWR, X2 BROSE-60-POL

Commit message: Some clean-ups
Parts:
- removed X2: BROSE-60-POL, con-panduit:057-060-1
- added D1, D10, D11, D12, D13, D14, D2, D3, D4, D5, D6, D7, D8, D9: BZV55, diode:ZENER-DIODESOD80C
- added JP1: (no value), pinhead:PINHD-1X55X2MM
- added LED3: A, adafruit:LEDSMT1206
- added R10, R11, R12, R13, R14, R15, R16, R17, R18, R19, R20, R21, R22, R9: 100K, rcl:R-EU_R1206
- added R7, R8: 150, rcl:R-EU_R1206
- added U15, U16: TD62783AP, uln-udn:UDN2981LW
- LED1: value A -> C
- R4: value 150 -> 10K
- X1: value PWR -> BROSE-60-POL; device adafruit:1X4-CLEANBIG -> con-panduit:057-060-1
Connections:
- removed net SR10_ROW15_24V: U10.7C, X2-15.S
- removed net SR11_ROW14_24V: U10.6C, X2-14.S
- removed net SR12_ROW13_24V: U10.5C, X2-13.S
- removed net SR13_ROW12_24V: U10.4C, X2-12.S
- removed net SR14_ROW11_24V: U10.3C, X2-11.S
- removed net SR15_ROW10_24V: U10.2C, X2-10.S
- removed net SR16_ROW9_24V: U10.1C, X2-9.S
- removed net SR17_ROW4_GND: U11.O4, U11.O5, U11.O6, U11.O7, U11.O8, X2-24.S
- removed net SR18_ROW3_GND: U11.O3, X2-23.S
- removed net SR19_ROW2_GND: U11.O2, X2-22.S
- removed net SR1_ROW8_24V: U9.8C, X2-8.S
- removed net SR20_ROW1_GND: U11.O1, X2-21.S
- removed net SR21_ROW20_24V: U14.8C, X2-20.S
- removed net SR22_ROW19_24V: U14.7C, X2-19.S
- removed net SR23_ROW18_24V: U14.6C, X2-18.S
- removed net SR24_ROW17_24V: U14.1C, U14.2C, U14.3C, U14.4C, U14.5C, X2-17.S
- removed net SR25_ROW12_GND: U12.O8, X2-32.S
- removed net SR26_ROW11_GND: U12.O7, X2-31.S
- removed net SR27_ROW10_GND: U12.O6, X2-30.S
- removed net SR28_ROW9_GND: U12.O5, X2-29.S
- removed net SR29_ROW8_GND: U12.O4, X2-28.S
- removed net SR2_ROW7_24V: U9.7C, X2-7.S
- removed net SR30_ROW7_GND: U12.O3, X2-27.S
- removed net SR31_ROW6_GND: U12.O2, X2-26.S
- removed net SR32_ROW5_GND: U12.O1, X2-25.S
- removed net SR33_ROW20_GND: U13.O8, X2-40.S
- removed net SR34_ROW19_GND: U13.O7, X2-39.S
- removed net SR35_ROW18_GND: U13.O6, X2-38.S
- removed net SR36_ROW17_GND: U13.O5, X2-37.S
- removed net SR37_ROW16_GND: U13.O4, X2-36.S
- removed net SR38_ROW15_GND: U13.O3, X2-35.S
- removed net SR39_ROW14_GND: U13.O2, X2-34.S
- removed net SR3_ROW6_24V: U9.6C, X2-6.S
- removed net SR40_ROW13_GND: U13.O1, X2-33.S
- removed net SR41_ADDR7: U7.QA, X2-59.S
- removed net SR42_ADDR6: U7.QB, X2-58.S
- removed net SR43_ADDR5: U7.QC, X2-57.S
- removed net SR44_ADDR4: U7.QD, X2-56.S
- removed net SR45_ADDR3: U7.QE, X2-55.S
- removed net SR46_ADDR2: U7.QF, X2-54.S
- removed net SR47_ADDR1: U7.QG, X2-53.S
- removed net SR48_B1@FP2800A: U7.QH, X2-52.S
- removed net SR49_B0@FP2800A: U8.QA, X2-51.S
- removed net SR4_ROW5_24V: U9.5C, X2-5.S
- removed net SR50_A2@FP2800A: U8.QB, X2-50.S
- removed net SR51_A1@FP2800A: U8.QC, X2-49.S
- removed net SR52_A0@FP2800A: U8.QD, X2-48.S
- removed net SR53_D@FP2800A: U8.QE, X2-47.S
- removed net SR54_ADDR8_NOT_EN: R5.1, U8.QF, X2-60.S
- removed net SR56_LED_A: R4.1, U8.QH
- removed net SR5_ROW4_24V: U9.4C, X2-4.S
- removed net SR6_ROW3_24V: U9.3C, X2-3.S
- removed net SR7_ROW2_24V: U9.2C, X2-2.S
- removed net SR8_ROW1_24V: U9.1C, X2-1.S
- removed net SR9_ROW16_24V: U10.8C, X2-16.S
- new net N$10: D6.C, R14.2
- new net N$12: D7.C, R15.2
- new net N$13: D8.C, R16.2
- new net N$14: D9.C, R17.2
- new net N$15: D10.C, R18.2
- new net N$16: D11.C, R19.2
- new net N$17: D12.C, R20.2
- new net N$18: D13.C, R21.2
- new net N$19: D14.C, R22.2
- new net N$2: D1.C, R9.2
- new net N$5: LED3.A, R8.2
- new net N$6: D2.C, R10.2
- new net N$7: D3.C, R11.2
- new net N$8: D4.C, R12.2
- new net N$9: D5.C, R13.2
- new net NOT_EN_ADDR8@FP2800A: MCU1.D1, R3.2, U15.I1, U15.I2, U15.I3
- new net NOT_EN_ADDR8@FP2800A_VS: R15.1, U15.O1, U15.O2, U15.O3, X1-60.S
- new net SR10_ROW10_SET: U12.O7, X1-10.S
- new net SR11_ROW11_SET: U12.O6, X1-11.S
- new net SR12_ROW12_SET: U12.O5, X1-12.S
- new net SR13_ROW13_SET: U12.O4, X1-13.S
- new net SR14_ROW14_SET: U12.O3, X1-14.S
- new net SR15_ROW15_SET: U12.O2, X1-15.S
- new net SR16_ROW16_SET: U12.O1, X1-16.S
- new net SR17_ROW17_SET: U11.O8, X1-17.S
- new net SR18_ROW18_SET: U11.O7, X1-18.S
- new net SR19_ROW19_SET: U11.O6, X1-19.S
- new net SR1_ROW1_SET: U13.O8, X1-1.S
- new net SR20_ROW20_SET: U11.O1, U11.O2, U11.O3, U11.O4, U11.O5, X1-20.S
- new net SR21_ROW1_RST: U14.4C, U14.5C, U14.6C, U14.7C, U14.8C, X1-21.S
- new net SR22_ROW2_RST: U14.3C, X1-22.S
- new net SR23_ROW3_RST: U14.2C, X1-23.S
- new net SR24_ROW4_RST: U14.1C, X1-24.S
- new net SR25_ROW5_RST: U10.8C, X1-25.S
- new net SR26_ROW6_RST: U10.7C, X1-26.S
- new net SR27_ROW7_RST: U10.6C, X1-27.S
- new net SR28_ROW8_RST: U10.5C, X1-28.S
- new net SR29_ROW9_RST: U10.4C, X1-29.S
- new net SR2_ROW2_SET: U13.O7, X1-2.S
- new net SR30_ROW10_RST: U10.3C, X1-30.S
- new net SR31_ROW11_RST: U10.2C, X1-31.S
- new net SR32_ROW12_RST: U10.1C, X1-32.S
- new net SR33_ROW13_RST: U9.8C, X1-33.S
- new net SR34_ROW14_RST: U9.7C, X1-34.S
- new net SR35_ROW15_RST: U9.6C, X1-35.S
- new net SR36_ROW16_RST: U9.5C, X1-36.S
- new net SR37_ROW17_RST: U9.4C, X1-37.S
- new net SR38_ROW18_RST: U9.3C, X1-38.S
- new net SR39_ROW19_RST: U9.2C, X1-39.S
- new net SR3_ROW3_SET: U13.O6, X1-3.S
- new net SR40_ROW20_RST: U9.1C, X1-40.S
- new net SR41_D@FP2800A: U16.I8, U7.QA
- new net SR41_D@FP2800A_VS: R22.1, U16.O8, X1-47.S
- new net SR42_A0@FP2800A: U16.I7, U7.QB
- new net SR42_A0@FP2800A_VS: R21.1, U16.O7, X1-48.S
- new net SR43_A1@FP2800A: U16.I6, U7.QC
- new net SR43_A1@FP2800A_VS: R20.1, U16.O6, X1-49.S
- new net SR44_A2@FP2800A: U16.I5, U7.QD
- new net SR44_A2@FP2800A_VS: R19.1, U16.O5, X1-50.S
- new net SR45_B0@FP2800A: U16.I4, U7.QE
- new net SR45_B0@FP2800A_VS: R18.1, U16.O4, X1-51.S
- new net SR46_B1@FP2800A: U16.I3, U7.QF
- new net SR46_B1@FP2800A_VS: R17.1, U16.O3, X1-52.S
- new net SR47_ADDR1@FP2800A: U16.I2, U7.QG
- new net SR47_ADDR1@FP2800A_VS: R14.1, U16.O2, X1-53.S
- new net SR48_ADDR2@FP2800A: U16.I1, U7.QH
- new net SR48_ADDR2@FP2800A_VS: R13.1, U16.O1, X1-54.S
- new net SR49_ADDR3@FP2800A: U15.I8, U8.QA
- new net SR49_ADDR3@FP2800A_VS: R12.1, U15.O8, X1-55.S
- new net SR4_ROW4_SET: U13.O5, X1-4.S
- new net SR50_ADDR4@FP2800A: U15.I7, U8.QB
- new net SR50_ADDR4@FP2800A_VS: R11.1, U15.O7, X1-56.S
- new net SR51_ADDR5@FP2800A: U15.I6, U8.QC
- new net SR51_ADDR5@FP2800A_VS: R10.1, U15.O6, X1-57.S
- new net SR52_ADDR6@FP2800A: U15.I5, U8.QD
- new net SR52_ADDR6@FP2800A_VS: R9.1, U15.O5, X1-58.S
- new net SR53_ADDR7@FP2800A: U15.I4, U8.QE
- new net SR53_ADDR7@FP2800A_VS: R16.1, U15.O4, X1-59.S
- new net SR54_LED_A: R8.1, U8.QF
- new net SR56_LED_C: R6.1, U8.QH
- new net SR5_ROW5_SET: U13.O4, X1-5.S
- new net SR6_ROW6_SET: U13.O3, X1-6.S
- new net SR7_ROW7_SET: U13.O2, X1-7.S
- new net SR8_ROW8_SET: U13.O1, X1-8.S
- new net SR9_ROW9_SET: U12.O8, X1-9.S
- net +24V: now also JP1.1, X1-42.S, X1-43.S; no longer X1.1, X2-42.S, X2-43.S
- net +3V3: now also JP1.3; no longer X1.3
- net +3V3_SW: now also R3.1, R4.1
- net +5V: now also JP1.2, R5.1, X1-45.S; no longer R3.1, R5.2, X1.2, X2-45.S
- net +VS: now also U15.VS, U16.VS, X1-44.S; no longer X2-44.S
- net EN_VS: now also JP1.4, MCU1.D4, R4.2; no longer MCU1.D3
- net GND: now also D1.A, D10.A, D11.A, D12.A, D13.A, D14.A, D2.A, D3.A, D4.A, D5.A, D6.A, D7.A, D8.A, D9.A, JP1.5, LED3.C, U15.GND, U16.GND, X1-41.S; no longer X1.4, X2-41.S
- net N$142: now also R7.2; no longer R6.2
- net N$148: now also R6.2; no longer R4.2
- net SR1: now also U13.I8; no longer U9.8B
- net SR10: now also U12.I7; no longer U10.7B
- net SR11: now also U12.I6; no longer U10.6B
- net SR12: now also U12.I5; no longer U10.5B
- net SR13: now also U12.I4; no longer U10.4B
- net SR14: now also U12.I3; no longer U10.3B
- net SR15: now also U12.I2; no longer U10.2B
- net SR16: now also U12.I1; no longer U10.1B
- net SR17: no longer U11.I4, U11.I5, U11.I6, U11.I7
- net SR18: now also U11.I7; no longer U11.I3
- net SR19: now also U11.I6; no longer U11.I2
- net SR2: now also U13.I7; no longer U9.7B
- net SR20: now also U11.I2, U11.I3, U11.I4, U11.I5
- net SR21: now also U14.4B, U14.5B, U14.6B, U14.7B
- net SR22: now also U14.3B; no longer U14.7B
- net SR23: now also U14.2B; no longer U14.6B
- net SR24: no longer U14.2B, U14.3B, U14.4B, U14.5B
- net SR25: now also U10.8B; no longer U12.I8
- net SR26: now also U10.7B; no longer U12.I7
- net SR27: now also U10.6B; no longer U12.I6
- net SR28: now also U10.5B; no longer U12.I5
- net SR29: now also U10.4B; no longer U12.I4
- net SR3: now also U13.I6; no longer U9.6B
- net SR30: now also U10.3B; no longer U12.I3
- net SR31: now also U10.2B; no longer U12.I2
- net SR32: now also U10.1B; no longer U12.I1
- net SR33: now also U9.8B; no longer U13.I8
- net SR34: now also U9.7B; no longer U13.I7
- net SR35: now also U9.6B; no longer U13.I6
- net SR36: now also U9.5B; no longer U13.I5
- net SR37: now also U9.4B; no longer U13.I4
- net SR38: now also U9.3B; no longer U13.I3
- net SR39: now also U9.2B; no longer U13.I2
- net SR4: now also U13.I5; no longer U9.5B
- net SR40: now also U9.1B; no longer U13.I1
- net SR5: now also U13.I4; no longer U9.4B
- net SR55_LED_B: now also R7.1; no longer R6.1
- net SR6: now also U13.I3; no longer U9.3B
- net SR7: now also U13.I2; no longer U9.2B
- net SR8: now also U13.I1; no longer U9.1B
- net SR9: now also U12.I8; no longer U10.8B
- net ~OE: now also R5.2; no longer R3.2
Other:
- note added: "24V logic level converter"
- note removed: "D3 with 10K pull-up"
- note removed: "D8 with 10K pull-down"
- moved on the sheet: C1, C2, J1, LED1, LED2, MCU1, R1, R2, R3, R4, R5, R6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

Commit message: Update board to rev10
Parts:
- removed D1, D10, D11, D12, D13, D14, D2, D3, D4, D5, D6, D7, D8, D9: BZV55, diode:ZENER-DIODESOD80C
- removed J1: INT_3V3, SparkFun-Connectors:M021X02_NO_SILK
- removed R10, R11, R12, R13, R14, R15, R16, R17, R18, R19, R20, R21, R22, R9: 100K, rcl:R-EU_R1206
- removed U15, U16: TD62783AP, uln-udn:UDN2981LW
- added C3: 22u, rcl:C-EUC1206
- added IC1: 74HCT245DW, 74xx-eu:74HCT245DW
- added IC16, IC17: ULN2803A, Texas Instruments_By_element14_Batch_1:ULN2803ADW
- added JP2: 24V, jumper:JP1E
- added JP3: 5V, jumper:JP1E
- added JP4: VS, jumper:JP1E
- added PAD1: 24V, wirepad:2,15/1,0
- added PAD2: VS, wirepad:2,15/1,0
- added X2: 5V, Rembrandt Electronics - JST XH Connectors v1-0:JST-XH-02-PIN-LONG-PAD
- added X3: 24V, Rembrandt Electronics - JST XH Connectors v1-0:JST-XH-02-PIN-LONG-PAD
- added X4: ~EN_PWR, Rembrandt Electronics - JST XH Connectors v1-0:JST-XH-02-PIN-LONG-PAD
- added X5: BROSE-60-POL, con-panduit:057-060-1
- C1: value 100u -> 100u/35V; device rcl:CPOL-EUC -> rcl:CPOL-EUE
- C2: value 22u -> 100u; device rcl:CPOL-EUB -> rcl:C-EUC1206
- IC10, IC11, IC12: value TD62783AP -> TD62783AFG
- IC13, IC14, IC15: value ULN2803ADW -> ULN2803A
- JP1: value (none) -> 3V3; device pinhead:PINHD-1X55X2MM -> jumper:JP1E
- LED1: value C -> C (red)
- LED2: value B -> B (yellow)
- LED3: value A -> A (green)
- R1: value 680K -> 470K
- R6: value 150 -> 180
- R8: value 150 -> 120
- X1: value BROSE-60-POL -> 3V3; device con-panduit:057-060-1 -> Rembrandt Electronics - JST XH Connectors v1-0:JST-XH-02-PIN-LONG-PAD
- renumbered U1 to IC2, U10 to IC14, U11 to IC10, U12 to IC11, U13 to IC12, U14 to IC15, U2 to IC3, U3 to IC4, U4 to IC5, U5 to IC6, U6 to IC7, U7 to IC8, U8 to IC9, U9 to IC13
Connections:
- removed net +24V: C1.+, IC2.VIN, JP1.1, R2.2, X1-42.S, X1-43.S
- removed net +3V3: J1.2, JP1.3
- removed net +3V3_SW: J1.1, MCU1.3V3, R3.1, R4.1
- removed net +5V: IC3.VCC, IC4.VCC, IC5.VCC, IC6.VCC, IC7.VCC, IC8.VCC, IC9.VCC, JP1.2, R5.1, X1-45.S
- removed net +VS: C2.+, IC10.VS, IC11.VS, IC12.VS, IC13.COM, IC14.COM, IC15.COM, IC2.VOUT, U15.VS, U16.VS, X1-44.S
- removed net EN_VS: IC2.ON, JP1.4, MCU1.D4, R4.2
- removed net N$10: D6.C, R14.2
- removed net N$12: D7.C, R15.2
- removed net N$13: D8.C, R16.2
- removed net N$14: D9.C, R17.2
- removed net N$142: LED2.A, R7.2
- removed net N$148: LED1.A, R6.2
- removed net N$15: D10.C, R18.2
- removed net N$16: D11.C, R19.2
- removed net N$17: D12.C, R20.2
- removed net N$18: D13.C, R21.2
- removed net N$19: D14.C, R22.2
- removed net N$2: D1.C, R9.2
- removed net N$6: D2.C, R10.2
- removed net N$7 (its old number): D3.C, R11.2
- removed net N$9: D5.C, R13.2
- removed net NOT_EN_ADDR8@FP2800A: MCU1.D1, R3.2, U15.I1, U15.I2, U15.I3
- removed net NOT_EN_ADDR8@FP2800A_VS: R15.1, U15.O1, U15.O2, U15.O3, X1-60.S
- removed net SR41_D@FP2800A_VS: R22.1, U16.O8, X1-47.S
- removed net SR42_A0@FP2800A_VS: R21.1, U16.O7, X1-48.S
- removed net SR43_A1@FP2800A_VS: R20.1, U16.O6, X1-49.S
- removed net SR44_A2@FP2800A_VS: R19.1, U16.O5, X1-50.S
- removed net SR45_B0@FP2800A_VS: R18.1, U16.O4, X1-51.S
- removed net SR46_B1@FP2800A_VS: R17.1, U16.O3, X1-52.S
- removed net SR47_ADDR1@FP2800A_VS: R14.1, U16.O2, X1-53.S
- removed net SR48_ADDR2@FP2800A_VS: R13.1, U16.O1, X1-54.S
- removed net SR49_ADDR3@FP2800A_VS: R12.1, U15.O8, X1-55.S
- removed net SR50_ADDR4@FP2800A_VS: R11.1, U15.O7, X1-56.S
- removed net SR51_ADDR5@FP2800A_VS: R10.1, U15.O6, X1-57.S
- removed net SR52_ADDR6@FP2800A_VS: R9.1, U15.O5, X1-58.S
- removed net SR53_ADDR7@FP2800A_VS: R16.1, U15.O4, X1-59.S
- new net 24V: IC16.COM, IC17.COM, JP2.1, X5-42.S, X5-43.S
- new net 24V_SW: C1.+, C2.1, IC2.VIN, JP2.2, PAD1.P, R2.2, X3-1.S
- new net 3V3: JP1.2, X1-1.S
- new net 3V3_SW: JP1.1, MCU1.3V3, R3.1
- new net N$21: LED2.C, R7.2
- new net N$23: LED3.C, R8.2
- new net RCLK_5V: IC1A.A6, IC3.RCLK, IC4.RCLK, IC5.RCLK, IC6.RCLK, IC7.RCLK, IC8.RCLK, IC9.RCLK
- new net SER_5V: IC1A.A4, IC3.SER
- new net SR41_D@FP2800A_24V: IC17.8C, X5-47.S
- new net SR42_A0@FP2800A_24V: IC17.7C, X5-48.S
- new net SR43_A1@FP2800A_24V: IC17.6C, X5-49.S
- new net SR44_A2@FP2800A_24V: IC17.5C, X5-50.S
- new net SR45_B0@FP2800A_24V: IC17.4C, X5-51.S
- new net SR46_B1@FP2800A_24V: IC17.3C, X5-52.S
- new net SR47_ADDR1@FP2800A_24V: IC17.2C, X5-53.S
- new net SR48_ADDR2@FP2800A_24V: IC17.1C, X5-54.S
- new net SR49_ADDR3@FP2800A_24V: IC16.6C, IC16.7C, IC16.8C, X5-55.S
- new net SR50_ADDR4@FP2800A_24V: IC16.5C, X5-56.S
- new net SR51_ADDR5@FP2800A_24V: IC16.4C, X5-57.S
- new net SR52_ADDR6@FP2800A_24V: IC16.3C, X5-58.S
- new net SR53_ADDR7@FP2800A_24V: IC16.2C, X5-59.S
- new net SRCLK_5V: IC1A.A7, IC3.SRCLK, IC4.SRCLK, IC5.SRCLK, IC6.SRCLK, IC7.SRCLK, IC8.SRCLK, IC9.SRCLK
- new net VCC: IC3.VCC, IC4.VCC, IC5.VCC, IC6.VCC, IC7.VCC, IC8.VCC, IC9.VCC, JP3.2, LED1.A, LED2.A, LED3.A, R4.1, R5.1, X2-1.S, X5-45.S
- new net VCC_SW: JP3.1, MCU1.5V
- new net VS: IC10.VS, IC11.VS, IC12.VS, IC13.COM, IC14.COM, IC15.COM, JP4.1, X5-44.S
- new net VS_SW: C3.1, IC2.VOUT, JP4.2, PAD2.P
- new net ~EN_ADDR8@FP2800A: IC1A.B1, IC1A.B2, IC1A.B3, MCU1.D3
- new net ~EN_ADDR8@FP2800A_24V: IC16.1C, X5-60.S
- new net ~EN_ADDR8@FP2800A_5V: IC16.1B, IC1A.A1, IC1A.A2, IC1A.A3, R4.2
- new net ~EN_POWER_RAILS: IC1A.DIR, IC1A.G, IC2.ON, MCU1.D1, R3.2, X4-1.S
- new net ~OE_5V: IC1A.A5, IC3.~OE, IC4.~OE, IC5.~OE, IC6.~OE, IC7.~OE, IC8.~OE, IC9.~OE, R5.2
- new net ~SRCLR_5V: IC1A.A8, IC3.~SRCLR, IC4.~SRCLR, IC5.~SRCLR, IC6.~SRCLR, IC7.~SRCLR, IC8.~SRCLR, IC9.~SRCLR
- net GND: now also C2.2, C3.2, IC16.GND, IC17.GND, X1-2.S, X2-2.S, X3-2.S, X4-2.S, X5-41.S; no longer C2.-, D1.A, D10.A, D11.A, D12.A, D13.A, D14.A, D2.A, D3.A, D4.A, D5.A, D6.A, D7.A, D8.A, D9.A, JP1.5, LED1.C, LED2.C, LED3.C, U15.GND, U16.GND, X1-41.S
- net N$5: now also LED1.C, R6.2; no longer LED3.A, R8.2
- net N$8: now also MCU1.D0, MCU1.RST; no longer D4.C, R12.2
- net RCLK: now also IC1A.B6; no longer IC3.RCLK, IC4.RCLK, IC5.RCLK, IC6.RCLK, IC7.RCLK, IC8.RCLK, IC9.RCLK
- net SER: now also IC1A.B4; no longer IC3.SER
- net SR10_ROW10_SET: now also X5-10.S; no longer X1-10.S
- net SR11_ROW11_SET: now also X5-11.S; no longer X1-11.S
- net SR12_ROW12_SET: now also X5-12.S; no longer X1-12.S
- net SR13_ROW13_SET: now also X5-13.S; no longer X1-13.S
- net SR14_ROW14_SET: now also X5-14.S; no longer X1-14.S
- net SR15_ROW15_SET: now also X5-15.S; no longer X1-15.S
- net SR16_ROW16_SET: now also X5-16.S; no longer X1-16.S
- net SR17_ROW17_SET: now also X5-17.S; no longer X1-17.S
- net SR18_ROW18_SET: now also X5-18.S; no longer X1-18.S
- net SR19_ROW19_SET: now also X5-19.S; no longer X1-19.S
- net SR1_ROW1_SET: now also X5-1.S; no longer X1-1.S
- net SR20_ROW20_SET: now also X5-20.S; no longer X1-20.S
- net SR21_ROW1_RST: now also X5-21.S; no longer X1-21.S
- net SR22_ROW2_RST: now also X5-22.S; no longer X1-22.S
- net SR23_ROW3_RST: now also X5-23.S; no longer X1-23.S
- net SR24_ROW4_RST: now also X5-24.S; no longer X1-24.S
- net SR25_ROW5_RST: now also X5-25.S; no longer X1-25.S
- net SR26_ROW6_RST: now also X5-26.S; no longer X1-26.S
- net SR27_ROW7_RST: now also X5-27.S; no longer X1-27.S
- net SR28_ROW8_RST: now also X5-28.S; no longer X1-28.S
- net SR29_ROW9_RST: now also X5-29.S; no longer X1-29.S
- net SR2_ROW2_SET: now also X5-2.S; no longer X1-2.S
- net SR30_ROW10_RST: now also X5-30.S; no longer X1-30.S
- net SR31_ROW11_RST: now also X5-31.S; no longer X1-31.S
- net SR32_ROW12_RST: now also X5-32.S; no longer X1-32.S
- net SR33_ROW13_RST: now also X5-33.S; no longer X1-33.S
- net SR34_ROW14_RST: now also X5-34.S; no longer X1-34.S
- net SR35_ROW15_RST: now also X5-35.S; no longer X1-35.S
- net SR36_ROW16_RST: now also X5-36.S; no longer X1-36.S
- net SR37_ROW17_RST: now also X5-37.S; no longer X1-37.S
- net SR38_ROW18_RST: now also X5-38.S; no longer X1-38.S
- net SR39_ROW19_RST: now also X5-39.S; no longer X1-39.S
- net SR3_ROW3_SET: now also X5-3.S; no longer X1-3.S
- net SR40_ROW20_RST: now also X5-40.S; no longer X1-40.S
- net SR41_D@FP2800A: now also IC17.8B; no longer U16.I8
- net SR42_A0@FP2800A: now also IC17.7B; no longer U16.I7
- net SR43_A1@FP2800A: now also IC17.6B; no longer U16.I6
- net SR44_A2@FP2800A: now also IC17.5B; no longer U16.I5
- net SR45_B0@FP2800A: now also IC17.4B; no longer U16.I4
- net SR46_B1@FP2800A: now also IC17.3B; no longer U16.I3
- net SR47_ADDR1@FP2800A: now also IC17.2B; no longer U16.I2
- net SR48_ADDR2@FP2800A: now also IC17.1B; no longer U16.I1
- net SR49_ADDR3@FP2800A: now also IC16.6B, IC16.7B, IC16.8B; no longer U15.I8
- net SR4_ROW4_SET: now also X5-4.S; no longer X1-4.S
- net SR50_ADDR4@FP2800A: now also IC16.5B; no longer U15.I7
- net SR51_ADDR5@FP2800A: now also IC16.4B; no longer U15.I6
- net SR52_ADDR6@FP2800A: now also IC16.3B; no longer U15.I5
- net SR53_ADDR7@FP2800A: now also IC16.2B; no longer U15.I4
- net SR5_ROW5_SET: now also X5-5.S; no longer X1-5.S
- net SR6_ROW6_SET: now also X5-6.S; no longer X1-6.S
- net SR7_ROW7_SET: now also X5-7.S; no longer X1-7.S
- net SR8_ROW8_SET: now also X5-8.S; no longer X1-8.S
- net SR9_ROW9_SET: now also X5-9.S; no longer X1-9.S
- net SRCLK: now also IC1A.B7; no longer IC3.SRCLK, IC4.SRCLK, IC5.SRCLK, IC6.SRCLK, IC7.SRCLK, IC8.SRCLK, IC9.SRCLK
- net ~OE: now also IC1A.B5; no longer IC3.~OE, IC4.~OE, IC5.~OE, IC6.~OE, IC7.~OE, IC8.~OE, IC9.~OE, R5.2
- net ~SRCLR: now also IC1A.B8, MCU1.D8; no longer IC3.~SRCLR, IC4.~SRCLR, IC5.~SRCLR, IC6.~SRCLR, IC7.~SRCLR, IC8.~SRCLR, IC9.~SRCLR, MCU1.D0
Other:
- note added: "24V GND logic level converter (to GND: inverting)"
- note added: "3V3 to 5V level shifter"
- note removed: "24V logic level converter"
- moved on the sheet: C1, LED1, LED2, LED3, R1, R3, R4
